File: AIFryer.kicad_pcb (KiCad board)
At the start: 2 copper layers, 100 x 56 mm, 39 parts, among them J1 KType, J3 ESPUartConn, J4 POWER, J5 ACIN, J6 ACIN, J7 ACIN, Q1 BTA16-600B, Q2 BTA16-600B, Q3 BSS126, U1 MAX6675, U3 ESP32-C3-WROOM-02-N4, U4 AMS1117-3.3, U5 MOC3021S, U6 4N25, U7 MOC3021S

Commit message: initial
Parts:
- removed C7: 100uF 10V Tant, Capacitor_Tantalum_SMD:CP_EIA-6032-28_Kemet-C
- removed HS1, HS2: Heatsink_Pad_2Pin, HeatsinkLibrary:Heatsink36x11
- removed J3: ESPUartConn, Connector_JST:JST_PH_B4B-PH-K_1x04_P2.00mm_Vertical
- removed J4: POWER, TerminalBlock_Phoenix:TerminalBlock_Phoenix_PT-1,5-2-3.5-H_1x02_P3.50mm_Horizontal
- removed U4: AMS1117-3.3, Package_TO_SOT_SMD:SOT-223-3_TabPin2
- added C10: 47n X2 2220, Capacitor_SMD:C_2220_5750Metric, F.Cu at (134.4, 141.0)
- added C11: 100n, Capacitor_SMD:C_0603_1608Metric, F.Cu at (97.7, 127.9)
- added C12: 100n, Capacitor_SMD:C_0603_1608Metric, F.Cu at (84.0, 128.4)
- added C18: 470u 10V, Capacitor_SMD:CP_Elec_6.3x7.7, F.Cu at (107.4, 107.0)
- added C2: 10n C0G, Capacitor_SMD:C_0603_1608Metric, F.Cu at (93.9, 138.4)
- added C6: 100n, Capacitor_SMD:C_0603_1608Metric, B.Cu at (103.6, 124.3)
- added D4: LED YG, LED_SMD:LED_0603_1608Metric, F.Cu at (131.4, 120.7)
- added D5: 1N5819WS, Diode_SMD:D_SOD-323, F.Cu at (103.5, 99.3)
- added D6: 1N5819WS, Diode_SMD:D_SOD-323, F.Cu at (147.4, 121.2)
- added D7: 1N5819WS, Diode_SMD:D_SOD-323, B.Cu at (76.9, 108.6)
- added F2: T500mA, Fuse:Fuse_Littelfuse_372_D8.50mm, F.Cu at (164.3, 119.3)
- added J10: DC IN, TerminalBlock_Phoenix:TerminalBlock_Phoenix_PT-1,5-2-3.5-H_1x02_P3.50mm_Horizontal, F.Cu at (74.6, 122.5)
- added J11: DC OUT, TerminalBlock_Phoenix:TerminalBlock_Phoenix_PT-1,5-2-3.5-H_1x02_P3.50mm_Horizontal, F.Cu at (74.6, 106.9)
- added J12: RELAY COM/NO/NC, TerminalBlock_Phoenix:TerminalBlock_Phoenix_PT-1,5-3-5.0-H_1x03_P5.00mm_Horizontal, F.Cu at (146.8, 148.5)
- added J2: K-TYPE, Connector_Phoenix_GMSTB:PhoenixContact_GMSTBA_2,5_2-G-7,62_1x02_P7.62mm_Horizontal, F.Cu at (77.8, 142.7)
- added J8: FAN, TerminalBlock_Phoenix:TerminalBlock_Phoenix_PT-1,5-2-5.0-H_1x02_P5.00mm_Horizontal, F.Cu at (134.3, 148.5)
- added J9: THERMAL FUSE, TerminalBlock_Phoenix:TerminalBlock_Phoenix_PT-1,5-2-5.0-H_1x02_P5.00mm_Horizontal, F.Cu at (164.2, 113.7)
- added JP1: VOUT SEL, Jumper:SolderJumper-3_P1.3mm_Open_RoundedPad1.0x1.5mm, F.Cu at (71.4, 116.2)
- added K1: SRD-05VDC-SL-C, Relay_THT:Relay_SPDT_SANYOU_SRD_Series_Form_C, F.Cu at (151.7, 124.8)
- added PS1: HLK-2M05 (5V 400mA), Converter_ACDC:Converter_ACDC_Hi-Link_HLK-2Mxx, F.Cu at (115.9, 107.0)
- added Q4: BTA16-600BW, Package_TO_SOT_THT:TO-220-3_Horizontal_TabUp, B.Cu at (134.5, 136.7)
- added Q5: AO3400A, Package_TO_SOT_SMD:SOT-23, B.Cu at (145.7, 123.1)
- added Q6: AO3400A, Package_TO_SOT_SMD:SOT-23, F.Cu at (74.6, 116.0)
- added R13: 10k, Resistor_SMD:R_0603_1608Metric, F.Cu at (105.8, 124.1)
- added R14: 180, Resistor_SMD:R_1206_3216Metric, B.Cu at (111.4, 141.4)
- added R15: 47, Resistor_SMD:R_1206_3216Metric, B.Cu at (105.4, 135.7)
- added R16: 10k, Resistor_SMD:R_0603_1608Metric, F.Cu at (118.6, 124.1)
- added R17: 180, Resistor_SMD:R_1206_3216Metric, B.Cu at (124.2, 141.4)
- added R18: 47, Resistor_SMD:R_1206_3216Metric, B.Cu at (118.2, 135.7)
- added R19: 10k, Resistor_SMD:R_0603_1608Metric, F.Cu at (131.4, 124.1)
- added R20: 390, Resistor_SMD:R_0603_1608Metric, F.Cu at (131.3, 122.5)
- added R21: 120, Resistor_SMD:R_0603_1608Metric, F.Cu at (131.5, 119.1)
- added R22: 180, Resistor_SMD:R_1206_3216Metric, F.Cu at (139.8, 141.5)
- added R23: 180, Resistor_SMD:R_1206_3216Metric, B.Cu at (137.0, 141.4)
- added R24: 47, Resistor_SMD:R_1206_3216Metric, B.Cu at (131.0, 140.4)
- added R25: 47, Resistor_SMD:R_1206_3216Metric, B.Cu at (131.0, 135.7)
- added R26: 10k, Resistor_SMD:R_0603_1608Metric, F.Cu at (88.7, 126.1)
- added R27: 10k, Resistor_SMD:R_0603_1608Metric, F.Cu at (91.2, 126.1)
- added R28: 100, Resistor_SMD:R_0603_1608Metric, F.Cu at (81.1, 123.0)
- added R29: 10k, Resistor_SMD:R_0603_1608Metric, F.Cu at (81.1, 125.5)
- added R30: 100, Resistor_SMD:R_0603_1608Metric, F.Cu at (77.7, 116.0)
- added R31: 10k, Resistor_SMD:R_0603_1608Metric, F.Cu at (77.0, 118.7)
- added R32: 10k, Resistor_SMD:R_0603_1608Metric, B.Cu at (103.6, 121.8)
- added R33: 10k, Resistor_SMD:R_0603_1608Metric, F.Cu at (93.7, 126.1)
- added RV1: 10D471K, Varistor:RV_Disc_D12mm_W4.2mm_P7.5mm, F.Cu at (148.0, 116.4)
- added TH1: 10k B3380, Resistor_SMD:R_0603_1608Metric, B.Cu at (104.4, 119.3)
- added TP1: +5V, TestPoint:TestPoint_THTPad_D1.5mm_Drill0.7mm, F.Cu at (57.7, 87.3)
- added TP2: +3.3V, TestPoint:TestPoint_THTPad_D1.5mm_Drill0.7mm, F.Cu at (57.7, 90.9)
- added TP3: GND, TestPoint:TestPoint_THTPad_D1.5mm_Drill0.7mm, F.Cu at (57.7, 94.4)
- added TP4: ZC, TestPoint:TestPoint_THTPad_D1.5mm_Drill0.7mm, F.Cu at (57.7, 98.0)
- added TP5: PWM_TOP, TestPoint:TestPoint_THTPad_D1.5mm_Drill0.7mm, F.Cu at (57.7, 101.5)
- added U2: MAX31856MUD+T, Package_SO:TSSOP-14_4.4x5mm_P0.65mm, F.Cu at (81.8, 134.0)
- added U8: MOC3052SR2M, Package_DIP:SMDIP-6_W9.53mm, F.Cu at (134.7, 130.5)
- C3: value 100n -> 10n C0G
- C4: moved to B.Cu
- C5: value 22u 25V -> 100n; footprint Capacitor_SMD:C_1206_3216Metric -> Capacitor_SMD:C_0603_1608Metric
- C8, C9: value 10n 400V -> 47n X2 2220; footprint Capacitor_THT:C_Rect_L13.0mm_W4.0mm_P10.00mm_FKS3_FKP3_MKS4 -> Capacitor_SMD:C_2220_5750Metric
- D1, D3: value LED -> LED YG
- J1: value KType -> K-TYPE
- J5: value ACIN -> AC IN
- J6: value ACIN -> HEATER TOP
- J7: value ACIN -> HEATER BOTTOM
- Q1, Q2: value BTA16-600B -> BTA16-600BW; footprint Package_TO_SOT_THT:TO-220-3_Vertical -> Package_TO_SOT_THT:TO-220-3_Horizontal_TabUp; moved to B.Cu
- R10: value 10k -> 47k
- R11, R5: value 1k -> 180; footprint Resistor_THT:R_Axial_DIN0309_L9.0mm_D3.2mm_P12.70mm_Horizontal -> Resistor_SMD:R_1206_3216Metric
- R12, R6: value 1k -> 47; footprint Resistor_THT:R_Axial_DIN0309_L9.0mm_D3.2mm_P12.70mm_Horizontal -> Resistor_SMD:R_1206_3216Metric; moved to B.Cu
- R2, R8: value 220 -> 120
- R3, R4: value 330 -> 390
- R7: value 2.2 -> 2.2k
- U1: value MAX6675 -> MAX31856MUD+T; footprint Package_SO:SOIC-8_3.9x4.9mm_P1.27mm -> Package_SO:TSSOP-14_4.4x5mm_P0.65mm
- U3: value ESP32-C3-WROOM-02-N4 -> ESP32-C3-SuperMini; footprint RF_Module:ESP32-C3-WROOM-02 -> AIFryer:ESP32-C3-SuperMini
- U5, U7: value MOC3021S -> MOC3052SR2M; footprint Package_DIP:DIP-6_W7.62mm_SMDSocket_SmallPads -> Package_DIP:SMDIP-6_W9.53mm
- U6: value 4N25 -> 4N25SR2M; footprint Package_DIP:DIP-6_W7.62mm_SMDSocket_SmallPads -> Package_DIP:SMDIP-6_W9.53mm; moved to B.Cu
- moved C4 69.1 mm to (138.6, 104.3)
- moved R6 42.4 mm to (105.4, 140.4), turned to 90 degrees
- moved Q1 41.8 mm to (108.9, 136.7), turned to 0 degrees
- moved R3 35.5 mm to (105.7, 122.5), turned to 0 degrees
- moved C8 34.7 mm to (108.8, 141.0), turned to 180 degrees
- moved U5 34.6 mm to (109.1, 130.5)
- moved D1 34.1 mm to (105.8, 120.7), turned to 0 degrees
- moved R2 33.4 mm to (105.9, 119.1), turned to 0 degrees
- moved J6 31.1 mm to (108.7, 148.5)
- moved R5 26.5 mm to (114.2, 141.5)
- moved R10 22.7 mm to (148.4, 108.5)
- moved J5 22.0 mm to (164.3, 135.2)
- moved R11 18.6 mm to (127.0, 141.5)
- moved U3 17.0 mm to (82.5, 99.3), turned to 0 degrees
- moved C3 14.6 mm to (80.2, 138.9), turned to 180 degrees
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Connections:
- C3 pad 1: Net-(U3-EN) -> /ThermoCouple2/TC+
- C3 pad 2: GND -> /ThermoCouple2/TC-
- C8 pad 1: AC-IN-L -> /L_HEAT
- C9 pad 1: AC-IN-L -> /L_HEAT
- D1 pad 2: PWM1 -> /PWM_TOP
- D3 pad 2: PWM2 -> /PWM_BOTTOM
- J1 pad 1: Net-(J1-Pin_1) -> /ThermoCouple1/TC-
- J1 pad 2: Net-(J1-Pin_2) -> /ThermoCouple1/TC+
- J6 pad 1: /TriacModule/LOAD -> /LOAD_TOP
- J7 pad 1: /TriacModule1/LOAD -> /LOAD_BOTTOM
- Q1 pad 1: /TriacModule/LOAD -> /LOAD_TOP
- Q1 pad 2: AC-IN-L -> /L_HEAT
- Q2 pad 1: /TriacModule1/LOAD -> /LOAD_BOTTOM
- Q2 pad 2: AC-IN-L -> /L_HEAT
- R1 pad 1: Net-(U3-EN) -> +3.3V
- R1 pad 2: +3.3V -> /MISO
- R10 pad 2: /ZeroCrossDetection/ZC -> /ZC
- R11 pad 2: AC-IN-L -> Net-(R11-Pad2)
- R12 pad 1: /TriacModule1/LOAD -> Net-(C9-Pad2)
- R12 pad 2: Net-(C9-Pad2) -> Net-(R12-Pad2)
- R2 pad 1: PWM1 -> /PWM_TOP
- R5 pad 2: AC-IN-L -> Net-(R14-Pad1)
- R6 pad 1: /TriacModule/LOAD -> Net-(C8-Pad2)
- R6 pad 2: Net-(C8-Pad2) -> Net-(R15-Pad1)
- R8 pad 1: PWM2 -> /PWM_BOTTOM
- U1 pad 2: Net-(J1-Pin_2) -> /ThermoCouple1/TC-
- U1 pad 3: Net-(J1-Pin_1) -> /ThermoCouple1/TC-
- U1 pad 4: +3.3V -> /ThermoCouple1/TC+
- U1 pad 5: SCK -> +3.3V
- U1 pad 6: CS1 -> unconnected-(U1-DNC-Pad6)
- U1 pad 7: MISO -> unconnected-(U1-~{DRDY}-Pad7)
- U1 pad 8: unconnected-(U1-NC-Pad8) -> +3.3V
- U3 pad 1: +3.3V -> /+5V_MCU
- U3 pad 10: unconnected-(U3-IO10-Pad10) -> /PWM_BOTTOM
- U3 pad 11: ESP RX -> /PWM_FAN
- U3 pad 12: ESP TX -> /CS1
- U3 pad 13: ZC1 -> /CS2
- U3 pad 14: PWM1 -> /RELAY
- U3 pad 15: CS2 -> /TC_FAULT
- U3 pad 16: SCK -> /MOSI
- U3 pad 2: Net-(U3-EN) -> GND
- U3 pad 3: CS1 -> +3.3V
- U3 pad 4: MOSI -> /SCK
- U3 pad 5: MISO -> /PWM_TOP
- U3 pad 6: ZC2 -> /MISO
- U3 pad 7: PWM2 -> /ZC
- U3 pad 8: ESP IO9 -> /NTC_ADC
- U3 pad 9: GND -> /DC_OUT
- U6 pad 5: /ZeroCrossDetection/ZC -> /ZC
Other:
- outline, holes or cut-outs redrawn
