File: AIFryer.kicad_sch (KiCad schematic)
At the start: 15 parts, among them J1 KType, J3 ESPUartConn, J4 POWER, J5 ACIN, J6 ACIN, J7 ACIN, U1 MAX6675, U3 ESP32-C3-WROOM-02-N4, U4 AMS1117-3.3

Commit message: initial
Parts:
- removed C7: 100uF 10V Tant, Capacitor_Tantalum_SMD:CP_EIA-6032-28_Kemet-C, symbol Device:C_Polarized_US
- removed J3: ESPUartConn, Connector_JST:JST_PH_B4B-PH-K_1x04_P2.00mm_Vertical, symbol Connector_Generic:Conn_01x04
- removed J4: POWER, TerminalBlock_Phoenix:TerminalBlock_Phoenix_PT-1,5-2-3.5-H_1x02_P3.50mm_Horizontal, symbol Connector:Screw_Terminal_01x02
- removed U3: ESP32-C3-WROOM-02-N4, RF_Module:ESP32-C3-WROOM-02, symbol GigaVescSymbols:ESP32-C3-WROOM-02-N4
- removed U4: AMS1117-3.3, Package_TO_SOT_SMD:SOT-223-3_TabPin2, symbol Regulator_Linear:AMS1117-3.3
- added C11, C12, C6: 100n, Capacitor_SMD:C_0603_1608Metric, symbol Device:C
- added C2: 10n C0G, Capacitor_SMD:C_0603_1608Metric, symbol Device:C
- added D5, D6, D7: 1N5819WS, Diode_SMD:D_SOD-323, symbol Diode:1N5819WS
- added F2: T500mA, Fuse:Fuse_Littelfuse_372_D8.50mm, symbol Device:Fuse
- added J10: DC IN, TerminalBlock_Phoenix:TerminalBlock_Phoenix_PT-1,5-2-3.5-H_1x02_P3.50mm_Horizontal, symbol Connector:Screw_Terminal_01x02
- added J11: DC OUT, TerminalBlock_Phoenix:TerminalBlock_Phoenix_PT-1,5-2-3.5-H_1x02_P3.50mm_Horizontal, symbol Connector:Screw_Terminal_01x02
- added J2: K-TYPE 2, Connector_Phoenix_GMSTB:PhoenixContact_GMSTBA_2,5_2-G-7,62_1x02_P7.62mm_Horizontal, symbol Connector_Generic:Conn_01x02
- added J8: FAN, TerminalBlock_Phoenix:TerminalBlock_Phoenix_PT-1,5-2-5.0-H_1x02_P5.00mm_Horizontal, symbol Connector_Generic:Conn_01x02
- added J9: THERMAL FUSE, TerminalBlock_Phoenix:TerminalBlock_Phoenix_PT-1,5-2-5.0-H_1x02_P5.00mm_Horizontal, symbol Connector_Generic:Conn_01x02
- added JP1: VOUT SEL, Jumper:SolderJumper-3_P1.3mm_Open_RoundedPad1.0x1.5mm, symbol Jumper:SolderJumper_3_Open
- added K1: SRD-05VDC-SL-C, Relay_THT:Relay_SPDT_SANYOU_SRD_Series_Form_C, symbol Relay:SANYOU_SRD_Form_C
- added PS1: HLK-5M05 (5V 1A), Converter_ACDC:Converter_ACDC_Hi-Link_HLK-5Mxx, symbol Converter_ACDC:HLK-5M05
- added Q5, Q6: AO3400A, Package_TO_SOT_SMD:SOT-23, symbol Transistor_FET:AO3400A
- added R26, R27, R29, R31, R32, R33: 10k, Resistor_SMD:R_0603_1608Metric, symbol Device:R
- added R28, R30: 100, Resistor_SMD:R_0603_1608Metric, symbol Device:R
- added RV1: 10D471K, Varistor:RV_Disc_D12mm_W4.2mm_P7.5mm, symbol Device:Varistor
- added TH1: 10k B3380, Resistor_SMD:R_0603_1608Metric, symbol Device:Thermistor_NTC
- added TP1: +5V, TestPoint:TestPoint_THTPad_D1.5mm_Drill0.7mm, symbol Connector:TestPoint
- added TP2: +3.3V, TestPoint:TestPoint_THTPad_D1.5mm_Drill0.7mm, symbol Connector:TestPoint
- added TP3: GND, TestPoint:TestPoint_THTPad_D1.5mm_Drill0.7mm, symbol Connector:TestPoint
- added TP4: ZC, TestPoint:TestPoint_THTPad_D1.5mm_Drill0.7mm, symbol Connector:TestPoint
- added TP5: PWM_TOP, TestPoint:TestPoint_THTPad_D1.5mm_Drill0.7mm, symbol Connector:TestPoint
- added U2: MAX31856MUD+T, Package_SO:TSSOP-14_4.4x5mm_P0.65mm, symbol Sensor_Temperature:MAX31856
- added U3: ESP32-C3-SuperMini, AIFryer:ESP32-C3-SuperMini, symbol AIFryer:ESP32-C3-SuperMini
- C1: LCSC Part # (none) -> C14663; MPN C14663 -> (none)
- C3: LCSC Part # (none) -> C14663; MPN C14663 -> (none); now not fitted
- C4: MPN C12891 -> (none)
- C5: value 22u 25V -> 10n C0G; footprint Capacitor_SMD:C_1206_3216Metric -> Capacitor_SMD:C_0603_1608Metric; MPN C12891 -> (none); now not fitted
- J1: value KType -> K-TYPE 1
- J5: value ACIN -> AC IN
- J6: value ACIN -> HEATER TOP; LCSC Part # (none) -> C5188434
- J7: value ACIN -> HEATER BOTTOM; LCSC Part # (none) -> C5188434
- R1: LCSC Part # (none) -> C25804; MPN C25804 -> (none)
- U1: value MAX6675 -> MAX31856MUD+T; footprint Package_SO:SOIC-8_3.9x4.9mm_P1.27mm -> Package_SO:TSSOP-14_4.4x5mm_P0.65mm; symbol MAXLibrary:MAX6675 -> Sensor_Temperature:MAX31856; LCSC Part # (none) -> C2653162
Connections:
- net +3.3V: now also C3.1, R1.1, U1.5 (AVDD), U1.8 (DVDD), C11.1, C12.1, R26.1, R27.1, R32.1, R33.1, TP2.1, U2.5 (AVDD), U2.8 (DVDD), U3.3 (3V3); no longer C5.1, R1.2, U1.4 (VCC)
- net +5V: now also D5.2 (A), D6.1 (K), JP1.1 (A), K1.5, PS1.4 (+Vout), TP1.1
- net AC-IN-L: now also F2.1, K1.1
- net AC-IN-N: now also J8.2 (Pin_2), PS1.2 (AC/N), RV1.2
- net CS1: now also U1.9 (~{CS}), R26.2, U3.12 (GPIO8); no longer U1.6 (~{CS})
- net CS2: now also R27.2, U2.9 (~{CS}), U3.13 (GPIO9)
- net GND: now also U1.14 (DGND), C11.2, C12.2, C6.2, J10.2 (Pin_2), PS1.3 (-Vout), Q5.2 (S), Q6.2 (S), R29.2, R31.2, TH1.2, TP3.1, U2.1 (AGND), U2.14 (DGND), U3.2 (GND); no longer C5.2
- net MISO: now also R1.2, U1.11 (SDO), U2.11 (SDO), U3.6 (GPIO2); no longer U1.7 (SO)
- net MOSI: now also U1.12 (SDI), U2.12 (SDI), U3.16 (GPIO21)
- net SCK: now also U1.10 (SCK), U2.10 (SCK), U3.4 (GPIO4); no longer U1.5 (SCK)
- net TC1+: now reaches J1.1 (Pin_1)
- net TC1+: now also U1.4 (T+), C2.1; no longer U1.3 (T+)
- net TC1-: now reaches J1.2 (Pin_2), U1.2 (BIAS)
- net TC1-: now also U1.3 (T-), C2.2
- net Triac_Top/LOAD renamed LOAD_TOP
- net Triac_Bottom/LOAD renamed LOAD_BOTTOM
- new net +5V_MCU: D5.1 (K), U3.1 (5V)
- new net DC_G: Q6.1 (G), R30.2, R31.1
- new net DC_OUT: R30.1, U3.9 (GPIO5)
- new net DC_SW: D7.2 (A), J11.2 (Pin_2), Q6.3 (D)
- new net LOAD_FAN: J8.1 (Pin_1)
- new net L_HEAT: J9.2 (Pin_2)
- new net L_PSU: F2.2, PS1.1 (AC/L), RV1.1
- new net L_RELAY: J9.1 (Pin_1), K1.3
- new net NTC_ADC: C6.1, R32.2, TH1.1, U3.8 (GPIO0)
- new net PWM_BOTTOM: U3.10 (GPIO6)
- new net PWM_FAN: U3.11 (GPIO7)
- new net PWM_TOP: TP5.1, U3.5 (GPIO3)
- new net RELAY: R28.1, U3.14 (GPIO10)
- new net RELAY_COIL: D6.2 (A), K1.2, Q5.3 (D)
- new net RELAY_G: Q5.1 (G), R28.2, R29.1
- new net TC2+: C5.1, J2.1 (Pin_1), U2.4 (T+)
- new net TC2-: C5.2, J2.2 (Pin_2), U2.2 (BIAS), U2.3 (T-)
- new net TC_FAULT: R33.2, U1.13 (~{FAULT}), U2.13 (~{FAULT}), U3.15 (GPIO20)
- new net V_DC: D7.1 (K), J11.1 (Pin_1), JP1.2 (C)
- new net V_EXT: J10.1 (Pin_1), JP1.3 (B)
- new net ZC: TP4.1, U3.7 (GPIO1)
- no-connect marks 0 -> 3
Other:
- sheet TriacModule renamed Triac_Top
- sheet TriacModule1 renamed Triac_Bottom
- added sheet Triac_Fan (TriacModule.kicad_sch)
- sheet Triac_Bottom ports: added LINE; removed none
- sheet Triac_Top ports: added LINE; removed none
- note added: "AIFryer / reflow oven controller - ESP32-C3 SuperMini, 3 triac channels, relay, DC output"
- note added: "HEATER MASTER RELAY + THERMAL FUSE LOOP Fan triac is fed BEFORE the relay so the fan keeps running on a fault."
- note added: "HEATSINK NTC (place near triac heatsinks)"
- note added: "LOW-SIDE DC OUTPUT (fan / light), max 24 V JP1 selects onboard +5V or external DC IN"
- note added: "MAINS INPUT / 5V SUPPLY No onboard main fuse: fuse the mains input upstream (fused inlet / enclosure). RV1 sits behind F2 so a shorted varistor blows F2."
- note added: "MCU - ESP32-C3 SuperMini (verify pinout + row spacing!) Strapping pins GPIO2/8/9 used only for inputs / idle-high chip selects."
- note added: "TEST POINTS"
- note added: "THERMOCOUPLES - MAX31856 (T- must NOT be grounded; BIAS tied to T-) TC2 channel footprint only (DNP). FAULT outputs wired-OR to GPIO20."
- note added: "TRIAC CHANNELS"
- moved on the sheet: C1, C4, J1, J5, J6, J7

Commit message: rework
Parts:
- removed C1, C11, C12, C3: 100n, Capacitor_SMD:C_0603_1608Metric, symbol Device:C
- removed C2, C5: 10n C0G, Capacitor_SMD:C_0603_1608Metric, symbol Device:C
- removed J1: K-TYPE 1, Connector_Phoenix_GMSTB:PhoenixContact_GMSTBA_2,5_2-G-7,62_1x02_P7.62mm_Horizontal, symbol Connector_Generic:Conn_01x02
- removed J2: K-TYPE 2, Connector_Phoenix_GMSTB:PhoenixContact_GMSTBA_2,5_2-G-7,62_1x02_P7.62mm_Horizontal, symbol Connector_Generic:Conn_01x02
- removed U1, U2: MAX31856MUD+T, Package_SO:TSSOP-14_4.4x5mm_P0.65mm, symbol Sensor_Temperature:MAX31856
- added J12: RELAY COM/NO/NC, TerminalBlock_Phoenix:TerminalBlock_Phoenix_PT-1,5-3-5.0-H_1x03_P5.00mm_Horizontal, symbol Connector_Generic:Conn_01x03
Connections:
- net AC-IN-L: now also J9.1 (Pin_1); no longer K1.1
- net RELAY_NC: now reaches K1.4
- net RELAY_NC: now also J12.3 (Pin_3)
- net L_RELAY renamed RELAY_NO
- net RELAY_NO: now also J12.2 (Pin_2); no longer J9.1 (Pin_1)
- new net RELAY_COM: J12.1 (Pin_1), K1.1
- no-connect marks 3 -> 0
Other:
- added sheet ThermoCouple1 (ThermoCouple.kicad_sch)
- added sheet ThermoCouple2 (ThermoCouple.kicad_sch)
- note added: "RELAY OUTPUT (dry contacts on J12) + HEATER THERMAL-FUSE LOOP (J9) J12 is isolated from the board: use it for a light, or loop it in series with J9 to get a firmware-controlled heater disconnect. Without that, a shorted triac is only stopped by the thermal fuse."
- note added: "THERMOCOUPLES - MAX31856 (T- must NOT be grounded; BIAS tied to T-) FAULT outputs wired-OR to GPIO20."
- note removed: "HEATER MASTER RELAY + THERMAL FUSE LOOP Fan triac is fed BEFORE the relay so the fan keeps running on a fault."
- note removed: "THERMOCOUPLES - MAX31856 (T- must NOT be grounded; BIAS tied to T-) TC2 channel footprint only (DNP). FAULT outputs wired-OR to GPIO20."
- title: (none) -> AIFryer - Reflow Oven Controller
- moved on the sheet: C6, D5, D6, D7, F2, J10, J11, J5, J6, J7, J8, J9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

Commit message: initial
Parts:
- added C18: 470u 10V, Capacitor_SMD:CP_Elec_6.3x7.7, symbol Device:C_Polarized
- C4: MPN (none) -> C12891
- C6: LCSC Part # C14663 -> (none); MPN (none) -> C14663
- D5, D6, D7: LCSC Part # C191023 -> (none); MPN (none) -> C191023
- F2: MPN (none) -> C529783
- J10, J11: LCSC Part # C695629 -> (none); MPN (none) -> C695629
- J12: MPN (none) -> C5188435
- J5: MPN (none) -> C5188434
- J6, J7, J8, J9: LCSC Part # C5188434 -> (none); MPN (none) -> C5188434
- K1: MPN (none) -> C35449
- PS1: value HLK-5M05 (5V 1A) -> HLK-2M05 (5V 400mA); footprint Converter_ACDC:Converter_ACDC_Hi-Link_HLK-5Mxx -> Converter_ACDC:Converter_ACDC_Hi-Link_HLK-2Mxx; symbol Converter_ACDC:HLK-5M05 -> Converter_ACDC:HLK-2M05; LCSC Part # C209907 -> (none); MPN (none) -> C209909
- Q5, Q6: LCSC Part # C20917 -> (none); MPN (none) -> C20917
- R1, R26, R27, R29, R31, R32, R33: LCSC Part # C25804 -> (none); MPN (none) -> C25804
- R28, R30: LCSC Part # C22775 -> (none); MPN (none) -> C22775
- RV1: MPN (none) -> C8760
- TH1: LCSC Part # C13564 -> (none); MPN (none) -> C13564
Connections:
- net +5V: now also C18.1
- net GND: now also C18.2
Other:
- moved on the sheet: D6, D7, J10, J11, J12, J6, J7, J8, J9, JP1, K1, Q5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
