File: ThermoCouple.kicad_sch (KiCad schematic)
At the start: 5 parts, among them J1 K-TYPE 1, U1 MAX31856MUD+T

Commit message: initial
Parts:
- C1, C11: LCSC Part # C14663 -> (none); MPN (none) -> C14663
- C2: MPN (none) -> C22399611
- J1: value K-TYPE 1 -> K-TYPE; MPN (none) -> C395930
- U1: LCSC Part # C2653162 -> (none); MPN (none) -> C2653162
Connections:
- net TC+: now also J1.2 (Pin_2); no longer J1.1 (Pin_1)
- net TC-: now also J1.1 (Pin_1); no longer J1.2 (Pin_2)
Other:
- moved on the sheet: J1
Changed lines of the file:
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@@
 	(symbol
 		(lib_id "Connector_Generic:Conn_01x02")
-		(at 86.36 92.71 0)
-		(mirror y)
+		(at 86.36 95.25 180)
 		(unit 1)
 		(body_style 1)
@@
 		(dnp no)
 		(property "Reference" "J1"
-			(at 86.36 90.17 0)
-			(show_name no)
-			(do_not_autoplace no)
-			(effects
-				(font
-					(size 1.27 1.27)
-				)
-			)
-		)
-		(property "Value" "K-TYPE 1"
-			(at 86.36 99.06 0)
+			(at 86.36 97.79 0)
+			(show_name no)
+			(do_not_autoplace no)
+			(effects
+				(font
+					(size 1.27 1.27)
+				)
+			)
+		)
+		(property "Value" "K-TYPE"
+			(at 86.36 88.9 0)
 			(show_name no)
 			(do_not_autoplace no)
@@
 		)
 		(property "Footprint" "Connector_Phoenix_GMSTB:PhoenixContact_GMSTBA_2,5_2-G-7,62_1x02_P7.62mm_Horizontal"
-			(at 86.36 92.71 0)
-			(hide yes)
-			(show_name no)
-			(do_not_autoplace no)
-			(effects
-				(font
-					(size 1.27 1.27)
-				)
-			)
-		)
-		(property "Datasheet" ""
-			(at 86.36 92.71 0)
+			(at 86.36 95.25 0)
+			(hide yes)
+			(show_name no)
+			(do_not_autoplace no)
+			(effects
+				(font
+					(size 1.27 1.27)
+				)
+			)
+		)
+		(property "Datasheet" ""
+			(at 86.36 95.25 0)
 			(hide yes)
 			(show_name no)
@@
 		)
 		(property "Description" ""
-			(at 86.36 92.71 0)
+			(at 86.36 95.25 0)
+			(hide yes)
+			(show_name no)
+			(do_not_autoplace no)
+			(effects
+				(font
+					(size 1.27 1.27)
+				)
+			)
+		)
+		(property "MPN" "C395930"
+			(at 86.36 95.25 0)
 			(hide yes)
 			(show_name no)
@@
 			)
 		)
-		(property "LCSC Part #" "C2653162"
+		(property "MPN" "C2653162"
 			(at 129.54 93.98 0)
 			(hide yes)
@@
 			)
 		)
-		(property "LCSC Part #" "C14663"
+		(property "MPN" "C14663"
 			(at 139.7 64.77 0)
 			(hide yes)
@@
 			)
 		)
-		(property "LCSC Part #" "C14663"
+		(property "MPN" "C14663"
 			(at 151.13 64.77 0)
 			(hide yes)
@@
 			(at 100.33 93.98 0)
 			(hide yes)
+			(show_name no)
+			(do_not_autoplace no)
+			(effects
+				(font
+					(size 1.27 1.27)
+				)
+			)
+		)
+		(property "MPN" "C22399611"
+			(at 100.33 93.98 0)
+			(hide yes)
