File: TriacModule.kicad_sch (KiCad schematic)
At the start: 9 parts, among them Q1 BTA16-600B, U5 MOC3021S

Commit message: initial
Parts:
- added R13: 10k, Resistor_SMD:R_0603_1608Metric, symbol Device:R
- added R14: 180, Resistor_SMD:R_1206_3216Metric, symbol Device:R
- added R15: 47, Resistor_SMD:R_1206_3216Metric, symbol Device:R
- C8: value 10n 400V -> 47n X2 275VAC; now not fitted
- Q1: value BTA16-600B -> BTA16-600BW; symbol Triac_Thyristor:BTA16-600B -> Triac_Thyristor:BTA16-600BW
- R2: value 220 -> 120; LCSC Part # (none) -> C22787
- R3: value 330 -> 390; LCSC Part # (none) -> C23151
- R5: value 1k -> 180; footprint Resistor_THT:R_Axial_DIN0309_L9.0mm_D3.2mm_P12.70mm_Horizontal -> Resistor_SMD:R_1206_3216Metric
- R6: value 1k -> 47; footprint Resistor_THT:R_Axial_DIN0309_L9.0mm_D3.2mm_P12.70mm_Horizontal -> Resistor_SMD:R_1206_3216Metric; now not fitted
- U5: value MOC3021S -> MOC3052M; symbol Relay_SolidState:MOC3021M -> Relay_SolidState:MOC3052M
Connections:
- net GND: now also R13.2
- net LOAD: now also R15.2; no longer R6.1
- net PWM: now also R13.1
- net at C8.2: now also R6.1; no longer R6.2
- net AC-IN-L renamed LINE
- net LINE: now also R14.2; no longer R5.2
- new net: R15.1, R6.2
- new net: R14.1, R5.2
- no-connect marks 0 -> 2
Other:
- note added: "Triac channel (used 3x: top element, bottom element, fan) MOC3052M random-phase driver; zero-cross timing comes from firmware + ZC detector. Rg: 2x 180R 1206 pulse-rated (Panasonic ERJ-P08 / Vishay CRCW-HP) in series. Snubber (C + 2x 47R 1206) DNP for first test; populate if the fan channel misbehaves."
- moved on the sheet: D1, HS1, Q1, R2, R3, R5, U5

Commit message: rework
Other:
- title: (none) -> AIFryer - Triac Channel
- moved on the sheet: C8, D1, Q1, R13, R14, R15, R2, R3, R5, R6

Commit message: initial
Parts:
- C8: value 47n X2 275VAC -> 47n X2 2220; footprint Capacitor_THT:C_Rect_L13.0mm_W4.0mm_P10.00mm_FKS3_FKP3_MKS4 -> Capacitor_SMD:C_2220_5750Metric; MPN (none) -> C5331998
- D1: value LED -> LED YG; MPN (none) -> C2987554
- HS1: now not fitted; now left out of the parts list
- Q1: footprint Package_TO_SOT_THT:TO-220-3_Vertical -> Package_TO_SOT_THT:TO-220-3_Horizontal_TabUp; MPN (none) -> C87396
- R13: LCSC Part # C25804 -> (none); MPN (none) -> C25804
- R14, R5: MPN (none) -> C20166761
- R2: LCSC Part # C22787 -> (none); MPN (none) -> C22787
- R3: LCSC Part # C23151 -> (none); MPN (none) -> C23151
- U5: value MOC3052M -> MOC3052SR2M; footprint Package_DIP:DIP-6_W7.62mm_SMDSocket_SmallPads -> Package_DIP:SMDIP-6_W9.53mm; MPN (none) -> C19864
Changed lines of the file:
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@@
 			)
 		)
-		(property "LCSC Part #" "C23151"
+		(property "MPN" "C23151"
 			(at 72.39 118.11 0)
 			(hide yes)
@@
 			)
 		)
-		(property "Value" "MOC3052M"
+		(property "Value" "MOC3052SR2M"
 			(at 93.98 106.68 0)
 			(show_name no)
@@
 			)
 		)
-		(property "Footprint" "Package_DIP:DIP-6_W7.62mm_SMDSocket_SmallPads"
+		(property "Footprint" "Package_DIP:SMDIP-6_W9.53mm"
 			(at 93.98 100.33 0)
 			(hide yes)
@@
 		)
 		(property "Description" ""
+			(at 93.98 100.33 0)
+			(hide yes)
+			(show_name no)
+			(do_not_autoplace no)
+			(effects
+				(font
+					(size 1.27 1.27)
+				)
+			)
+		)
+		(property "MPN" "C19864"
 			(at 93.98 100.33 0)
 			(hide yes)
@@
 			)
 		)
-		(property "Value" "47n X2 275VAC"
+		(property "Value" "47n X2 2220"
 			(at 161.2424 92.71 0)
 			(show_name no)
@@
 			)
 		)
-		(property "Footprint" "Capacitor_THT:C_Rect_L13.0mm_W4.0mm_P10.00mm_FKS3_FKP3_MKS4"
+		(property "Footprint" "Capacitor_SMD:C_2220_5750Metric"
 			(at 151.13 91.44 0)
 			(hide yes)
@@
 			)
 		)
-		(property "Description" ""
+		(property "Description" "X2 safety MLCC 250VAC (Fenghua FH20X473K302EHQ). Keep away from board edges / screws: a cracked MLCC fails short."
+			(at 151.13 91.44 0)
+			(hide yes)
+			(show_name no)
+			(do_not_autoplace no)
+			(effects
+				(font
+					(size 1.27 1.27)
+				)
+			)
+		)
+		(property "MPN" "C5331998"
 			(at 151.13 91.44 0)
 			(hide yes)
@@
 			)
 		)
-		(property "LCSC Part #" "C25804"
+		(property "MPN" "C25804"
 			(at 63.5 105.41 0)
 			(hide yes)
@@
 			)
 		)
+		(property "MPN" "C20166761"
+			(at 110.49 92.71 0)
+			(hide yes)
+			(show_name no)
+			(do_not_autoplace no)
+			(effects
+				(font
+					(size 1.27 1.27)
+				)
+			)
+		)
 		(pin "1"
 		)
@@
 			)
 		)
-		(property "Footprint" "Package_TO_SOT_THT:TO-220-3_Vertical"
+		(property "Footprint" "Package_TO_SOT_THT:TO-220-3_Horizontal_TabUp"
 			(at 129.54 100.33 0)
 			(hide yes)
@@
 		)
 		(property "Description" ""
+			(at 129.54 100.33 0)
+			(hide yes)
+			(show_name no)
+			(do_not_autoplace no)
+			(effects
+				(font
+					(size 1.27 1.27)
+				)
+			)
+		)
+		(property "MPN" "C87396"
 			(at 129.54 100.33 0)
 			(hide yes)
@@
 			)
 		)
-		(property "Value" "LED"
+		(property "Value" "LED YG"
 			(at 77.5176 105.41 90)
 			(show_name no)
@@
 		(property "Description" ""
 			(at 72.39 104.14 90)
+			(hide yes)
+			(show_name no)
+			(do_not_autoplace no)
+			(effects
+				(font
+					(size 1.27 1.27)
+				)
+			)
+		)
+		(property "MPN" "C2987554"
+			(at 72.39 104.14 0)
 			(hide yes)
 			(show_name no)
@@
 			)
 		)
-		(property "LCSC Part #" "C22787"
+		(property "MPN" "C22787"
 			(at 78.74 97.79 90)
 			(hide yes)
@@
 			)
 		)
+		(property "MPN" "C20166761"
+			(at 120.65 92.71 0)
+			(hide yes)
+			(show_name no)
+			(do_not_autoplace no)
+			(effects
+				(font
+					(size 1.27 1.27)
+				)
+			)
+		)
 		(pin "1"
 		)
@@
 		(body_style 1)
 		(exclude_from_sim no)
-		(in_bom yes)
-		(on_board yes)
-		(in_pos_files yes)
-		(dnp no)
+		(in_bom no)
+		(on_board no)
+		(in_pos_files no)
+		(dnp yes)
 		(property "Reference" "HS1"
 			(at 147.32 64.77 0)
