File: ZeroCrossDetection.kicad_sch (KiCad schematic)
At the start: 6 parts, among them Q3 BSS126, U6 4N25

Commit message: initial
Parts:
- R10: value 10k -> 47k
- R7: value 2.2 -> 2.2k
- U6: footprint Package_DIP:DIP-6_W7.62mm_SMDSocket_SmallPads -> Package_DIP:DIP-6_W7.62mm

Commit message: rework
Other:
- title: (none) -> AIFryer - Zero-Cross Detector
Changed lines of the file:
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@@
 	(generator_version "10.0")
 	(paper "A4")
+	(title_block
+		(title "AIFryer - Zero-Cross Detector")
+		(date "2026-10-02")
+		(rev "1")
+		(comment 1 "ABS6 bridge + BSS126 current source + 4N25")
+		(comment 2 "Output: ZC (active low pulse near zero crossing)")
+	)
 	(junction
 		(at 152.4 101.6)

Commit message: initial
Parts:
- D2: MPN (none) -> C54444726
- R10: MPN (none) -> C25819
- R7: MPN C22939 -> C4190
- U6: value 4N25 -> 4N25SR2M; footprint Package_DIP:DIP-6_W7.62mm -> Package_DIP:SMDIP-6_W9.53mm; MPN (none) -> C44165
Changed lines of the file:
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@@
+			)
+		)
+		(property "MPN" "C25819"
+			(at 190.5 86.36 0)
+			(hide yes)
+			(show_name no)
+			(do_not_autoplace no)
+			(effects
+				(font
+					(size 1.27 1.27)
+				)
 			)
 		)
@@
 			)
 		)
-		(property "MPN" "C22939"
+		(property "MPN" "C4190"
 			(at 152.4 95.25 0)
 			(hide yes)
@@
 			)
 		)
-		(property "Value" "4N25"
+		(property "Value" "4N25SR2M"
 			(at 177.8 88.9 0)
 			(show_name no)
@@
 			)
 		)
-		(property "Footprint" "Package_DIP:DIP-6_W7.62mm"
+		(property "Footprint" "Package_DIP:SMDIP-6_W9.53mm"
 			(at 172.72 100.33 0)
 			(hide yes)
@@
 		)
 		(property "Description" "DC Optocoupler Base Connected, Vce 30V, CTR 20%, Viso 2500V, DIP6"
+			(at 177.8 95.25 0)
+			(hide yes)
+			(show_name no)
+			(do_not_autoplace no)
+			(effects
+				(font
+					(size 1.27 1.27)
+				)
+			)
+		)
+		(property "MPN" "C44165"
 			(at 177.8 95.25 0)
 			(hide yes)
@@
 			(at 127 88.9 0)
 			(hide yes)
+			(show_name no)
+			(do_not_autoplace no)
+			(effects
+				(font
+					(size 1.27 1.27)
+				)
+			)
+		)
+		(property "MPN" "C54444726"
+			(at 127 88.9 0)
+			(hide yes)
